Commit message: Adds end-effector link/joint used in Isaac Sim

File: robots/common/franka_arm.xacro (robot description, xacro)
@@ -125,4 +125,11 @@
       <child link="${arm_id}_link8" />
     </joint>
+    <!-- Define the end_effector frame used in Isaac Sim -->
+    <link name="end_effector"/>
+    <joint name="end_effector_joint" type="fixed">
+      <xacro:franka-kinematics name="joint_ee" config="${kinematics}" />
+      <parent link="${arm_id}_hand" />
+      <child link="end_effector" />
+    </joint>
   </xacro:macro>
 </robot>

Commit message: Added draft values for the unscrewer

File: robots/common/franka_arm.xacro (robot description, xacro)
@@ -132,4 +132,43 @@
       <child link="end_effector" />
     </joint>
+        <!-- Unscrewer tool link -->
+    <link name="unscrewer">
+      <visual>
+        <geometry>
+          <!-- Use the unscrewer mesh -->
+          <mesh filename="package://franka_description/meshes/robot_arms/fr3/visual/unscrewer.dae" scale="1 1 1"/> <!-- Adjust the scale as necessary -->
+        </geometry>
+        <origin xyz="0 0 0" rpy="0 0 0.0"/>  <!-- Adjust the position of the unscrewer relative to the gripper 0 3.14159 0.785398163 -->
+        <material name="gray">
+          <color rgba="0.5 0.5 0.5 1"/>
+        </material>
+      </visual>
+      <collision>
+        <!-- First cylinder (larger one) with radius 0.01575 m and length 104.8 mm -->
+        <geometry>
+          <cylinder radius="0.01575" length="0.1048"/>
+        </geometry>
+        <origin xyz="0 0 -0.0524" rpy="0 0 0"/> <!-- Positioning to place it in the lower part-->
+      </collision>
+      <collision>
+        <!-- Second cylinder (smaller one) with radius 0.0385 m and length 104.8 mm -->
+        <geometry>
+          <cylinder radius="0.0385" length="0.085"/>
+        </geometry>
+        <origin xyz="0 0 -0.1473" rpy="0 0 0"/> <!-- Positioned to stack on top of the first cylinder -->
+      </collision>
+      <inertial>
+        <mass value="0.264659"/> <!-- Updated mass of the unscrewer -->
+        <origin xyz="-0.00000023 0.0000002276 -0.09747" rpy="0 0 0"/> <!-- Updated center of mass, converted to meters 0 3.14159 0.785398163 -->
+        <inertia ixx="0.000461783" ixy="0" ixz="0" iyy="0.000446552" iyz="-0.000000005" izz="0.000047542"/>
+      </inertial>
+    </link>
+    <!-- Fixed joint to attach unscrewer to link8 -->
+    <joint name="unscrewer_joint" type="fixed">
+      <xacro:franka-kinematics name="joint_unscrewer" config="${kinematics}" />
+      <parent link="${arm_id}_link8"/>
+      <child link="unscrewer"/>
+      <origin xyz="0 0 0.2407953" rpy="0 0 ${-pi/4}"/>
+    </joint>
   </xacro:macro>
 </robot>

Commit message: Adds values to inertials.yaml and brings back the franka_arm.xacro as we need it

File: robots/common/franka_arm.xacro (robot description, xacro)
@@ -132,5 +132,11 @@
       <child link="end_effector" />
     </joint>
-        <!-- Unscrewer tool link -->
+    <link name="end_effector_unscrewer_reach_test"/>
+    <joint name="end_effector_unscrewer_reach_test_joint" type="fixed">
+      <xacro:franka-kinematics name="joint_end_effector_unscrewer_reach_test" config="${kinematics}" />
+      <parent link="${arm_id}_hand" />
+      <child link="end_effector_unscrewer_reach_test" />
+    </joint>
+    <!-- Unscrewer tool link -->
     <link name="unscrewer">
       <visual>

Commit message: Removes end-effector from the joints and links

File: robots/common/franka_arm.xacro (robot description, xacro)
@@ -125,11 +125,4 @@
       <child link="${arm_id}_link8" />
     </joint>
-    <!-- Define the end_effector frame used in Isaac Sim -->
-    <link name="end_effector"/>
-    <joint name="end_effector_joint" type="fixed">
-      <xacro:franka-kinematics name="joint_ee" config="${kinematics}" />
-      <parent link="${arm_id}_hand" />
-      <child link="end_effector" />
-    </joint>
   </xacro:macro>
 </robot>

Commit message: feat: modified the collisons to be capsules

File: robots/common/franka_arm.xacro (robot description, xacro)
@@ -107,6 +107,4 @@
     <xacro:link_with_sc name="link7" gazebo="${gazebo}" rpy="0 0 ${pi/4}" with_sc="${with_sc}">
       <self_collision_geometries>
-        <xacro:collision_capsule xyz="0 0 0.01" direction="z" radius="${0.04+safety_distance}" length="0.14" />
-        <xacro:collision_capsule xyz="0.06 0 0.082" direction="x" radius="${0.03+safety_distance}"  length="0.01" />
       </self_collision_geometries>
     </xacro:link_with_sc>
@@ -136,21 +134,7 @@
         </material>
       </visual>
-      <collision>
-        <geometry>
-          <cylinder radius="0.01575" length="0.1048"/>
-        </geometry>
-        <origin xyz="0 0 -0.0524" rpy="0 0 0"/>
-      </collision>
-      <collision>
-        <geometry>
-          <cylinder radius="0.0385" length="0.085"/>
-        </geometry>
-        <origin xyz="0 0 -0.1473" rpy="0 0 0"/>
-      </collision>
-      <inertial>
-        <mass value="0.264659"/>
-        <origin xyz="-0.00000023 0.0000002276 -0.09747" rpy="0 0 0"/>
-        <inertia ixx="0.000461783" ixy="0" ixz="0" iyy="0.000446552" iyz="-0.000000005" izz="0.000047542"/>
-      </inertial>
+        <xacro:collision_capsule xyz="0 0 -0.149" direction="z" radius="0.044" length="0.045" />
+        <xacro:collision_capsule xyz="0 0 -0.05" direction="z" radius="0.02" length="0.065" />
+        <xacro:franka-inertials name="link_unscrewer" inertials="${inertials}" />
     </link>
     <joint name="unscrewer_joint" type="fixed">
@@ -169,15 +153,6 @@
         </material>
       </visual>
-      <collision>
-        <geometry>
-          <cylinder radius="0.027" length="0.20993"/>
-        </geometry>
-        <origin xyz="0 0 -0.104965" rpy="0 0 0"/>
-      </collision>
-      <inertial>
-        <mass value="0.178"/>
-        <origin xyz="-0.005423 0.000141 -0.097517" rpy="0 0 0"/>
-        <inertia ixx="0.000934085" ixy="0.000000103" ixz="-0.000064273" iyy="0.000938346" iyz="0.000001638" izz="0.000037901"/>
-      </inertial>
+        <xacro:collision_capsule xyz="0 0 -0.085" direction="z" radius="0.026" length="0.19" />
+        <xacro:franka-inertials name="link_camera" inertials="${inertials}" />
     </link>
     <joint name="camera_joint" type="fixed">

Commit message: changed how the links are made

File: robots/common/franka_arm.xacro (robot description, xacro)
@@ -107,4 +107,6 @@
     <xacro:link_with_sc name="link7" gazebo="${gazebo}" rpy="0 0 ${pi/4}" with_sc="${with_sc}">
       <self_collision_geometries>
+        <xacro:collision_capsule xyz="0 0 0.01" direction="z" radius="${0.04+safety_distance}" length="0.14" />
+        <xacro:collision_capsule xyz="0.06 0 0.082" direction="x" radius="${0.03+safety_distance}"  length="0.01" />
       </self_collision_geometries>
     </xacro:link_with_sc>
@@ -124,40 +126,24 @@
     </joint>
     <!-- Unscrewer tool link -->
-    <link name="unscrewer">
-      <visual>
-        <geometry>
-          <mesh filename="package://franka_description/meshes/robot_arms/fr3/visual/unscrewer.dae" scale="1 1 1"/>
-        </geometry>
-        <origin xyz="0 0 0" rpy="0 0 0.0"/>
-        <material name="gray">
-          <color rgba="0.5 0.5 0.5 1"/>
-        </material>
-      </visual>
-        <xacro:collision_capsule xyz="0 0 -0.149" direction="z" radius="0.044" length="0.045" />
-        <xacro:collision_capsule xyz="0 0 -0.05" direction="z" radius="0.02" length="0.065" />
-        <xacro:franka-inertials name="link_unscrewer" inertials="${inertials}" />
-    </link>
-    <joint name="unscrewer_joint" type="fixed">
-      <xacro:franka-kinematics name="joint_unscrewer" config="${kinematics}" />
+    <xacro:link_with_sc name="unscrewer" gazebo="${gazebo}" rpy="0 0 ${pi/4}" with_sc="${with_sc}">
+        <self_collision_geometries>
+          <xacro:collision_capsule xyz="0 0 -0.149" direction="z" radius="0.044" length="0.045" />
+          <xacro:collision_capsule xyz="0 0 -0.05" direction="z" radius="0.02" length="0.065" />
+        </self_collision_geometries>
+    </xacro:link_with_sc>
+    <joint name="unscrewer" type="fixed">
+      <xacro:franka-kinematics name="unscrewer" config="${kinematics}" />
       <parent link="${arm_id}_link8"/>
-      <child link="unscrewer"/>
+      <child link="${arm_id}_unscrewer"/>
     </joint>
-    <link name="camera">
-      <visual>
-        <geometry>
-          <mesh filename="package://franka_description/meshes/robot_arms/fr3/visual/camera.dae" scale="1 1 1"/>
-        </geometry>
-        <origin xyz="0 0 0" rpy="0 0 0"/>
-        <material name="white">
-          <color rgba="1 1 1 1"/>
-        </material>
-      </visual>
+    <xacro:link_with_sc name="camera" gazebo="${gazebo}" rpy="0 0 ${pi/4}" with_sc="${with_sc}">
+      <self_collision_geometries>
         <xacro:collision_capsule xyz="0 0 -0.085" direction="z" radius="0.026" length="0.19" />
-        <xacro:franka-inertials name="link_camera" inertials="${inertials}" />
-    </link>
-    <joint name="camera_joint" type="fixed">
-      <xacro:franka-kinematics name="joint_camera" config="${kinematics}" />
+      </self_collision_geometries>
+    </xacro:link_with_sc>
+    <joint name="camera" type="fixed">
+      <xacro:franka-kinematics name="camera" config="${kinematics}" />
       <parent link="${arm_id}_link8"/>
-      <child link="camera"/>
+      <child link="${arm_id}_camera"/>
     </joint>
   </xacro:macro>

Commit message: Adapts urdf sbtc additions according to new conventions

File: robots/common/franka_arm.xacro (robot description, xacro)
@@ -128,5 +128,5 @@
     </joint>
     <!-- Unscrewer tool link -->
-    <xacro:link_with_sc name="unscrewer" gazebo="${gazebo}" rpy="0 0 ${pi/4}" with_sc="${with_sc}">
+    <xacro:link_with_sc name="${prefix}unscrewer" gazebo="${gazebo}" rpy="0 0 ${pi/4}" with_sc="${with_sc}">
       <self_collision_geometries>
         <xacro:collision_capsule xyz="0 0 -0.149" direction="z" radius="${0.044+safety_distance}" length="0.045" />
@@ -134,18 +134,18 @@
       </self_collision_geometries>
     </xacro:link_with_sc>
-    <joint name="unscrewer" type="fixed">
+    <joint name="${prefix}unscrewer" type="fixed">
       <xacro:franka-kinematics name="unscrewer" config="${kinematics}" />
-      <parent link="${arm_id}_link8"/>
-      <child link="${arm_id}_unscrewer"/>
+      <parent link="${prefix}link8"/>
+      <child link="${prefix}unscrewer"/>
     </joint>
-    <xacro:link_with_sc name="camera" gazebo="${gazebo}" rpy="0 0 ${pi/4}" with_sc="${with_sc}">
+    <xacro:link_with_sc name="${prefix}camera" gazebo="${gazebo}" rpy="0 0 ${pi/4}" with_sc="${with_sc}">
       <self_collision_geometries>
         <xacro:collision_capsule xyz="0 0 -0.085" direction="z" radius="${0.026+safety_distance}" length="0.19" />
       </self_collision_geometries>
     </xacro:link_with_sc>
-    <joint name="camera" type="fixed">
+    <joint name="${prefix}camera" type="fixed">
       <xacro:franka-kinematics name="camera" config="${kinematics}" />
-      <parent link="${arm_id}_link8"/>
-      <child link="${arm_id}_camera"/>
+      <parent link="${prefix}link8"/>
+      <child link="${prefix}camera"/>
     </joint>
   </xacro:macro>

Commit message: made to work with cumotio

File: robots/common/franka_arm.xacro (robot description, xacro)
@@ -128,5 +128,5 @@
     </joint>
     <!-- Unscrewer tool link -->
-    <xacro:link_with_sc name="${prefix}unscrewer" gazebo="${gazebo}" rpy="0 0 ${pi/4}" with_sc="${with_sc}">
+    <xacro:link_with_sc name="unscrewer" gazebo="${gazebo}" rpy="0 0 ${pi/4}" with_sc="${with_sc}">
       <self_collision_geometries>
         <xacro:collision_capsule xyz="0 0 -0.149" direction="z" radius="${0.044+safety_distance}" length="0.045" />
@@ -134,18 +134,18 @@
       </self_collision_geometries>
     </xacro:link_with_sc>
-    <joint name="${prefix}unscrewer" type="fixed">
+    <joint name="unscrewer" type="fixed">
       <xacro:franka-kinematics name="unscrewer" config="${kinematics}" />
       <parent link="${prefix}link8"/>
-      <child link="${prefix}unscrewer"/>
+      <child link="unscrewer"/>
     </joint>
-    <xacro:link_with_sc name="${prefix}camera" gazebo="${gazebo}" rpy="0 0 ${pi/4}" with_sc="${with_sc}">
+    <xacro:link_with_sc name="camera" gazebo="${gazebo}" rpy="0 0 ${pi/4}" with_sc="${with_sc}">
       <self_collision_geometries>
         <xacro:collision_capsule xyz="0 0 -0.085" direction="z" radius="${0.026+safety_distance}" length="0.19" />
       </self_collision_geometries>
     </xacro:link_with_sc>
-    <joint name="${prefix}camera" type="fixed">
+    <joint name="camera" type="fixed">
       <xacro:franka-kinematics name="camera" config="${kinematics}" />
       <parent link="${prefix}link8"/>
-      <child link="${prefix}camera"/>
+      <child link="camera"/>
     </joint>
   </xacro:macro>
