Commit message: fix: gazebo can be used with prefixes

File: robots/common/franka_arm.ros2_control.xacro (robot description, xacro)
@@ -59,5 +59,5 @@
       <xacro:configure_joint joint_name="${arm_prefix}${arm_id}_joint7" initial_position="${pi/4}"/>
       <xacro:if value="${gazebo and hand}">
-        <xacro:configure_joint joint_name="${arm_id}_finger_joint1" initial_position="0.0" />
+        <xacro:configure_joint joint_name="${arm_prefix}${arm_id}_finger_joint1" initial_position="0.0" />
       </xacro:if>
       <xacro:macro name="general_purpose_io" params="prefix command_interface index">

File: robots/common/franka_robot.xacro (robot description, xacro)
@@ -104,39 +104,39 @@
           <origin xyz="${xyz}" rpy="${rpy}" />
           <parent link="${parent}" />
-          <child  link="${arm_id}_link0" />
+          <child  link="${arm_prefix}${arm_id}_link0" />
         </joint>
       </xacro:if>
-      <xacro:gazebo-joint joint="${arm_id}_joint1" transmission="hardware_interface/PositionJointInterface" />
-      <xacro:gazebo-joint joint="${arm_id}_joint2" transmission="hardware_interface/PositionJointInterface" />
-      <xacro:gazebo-joint joint="${arm_id}_joint3" transmission="hardware_interface/PositionJointInterface" />
-      <xacro:gazebo-joint joint="${arm_id}_joint4" transmission="hardware_interface/PositionJointInterface" />
-      <xacro:gazebo-joint joint="${arm_id}_joint5" transmission="hardware_interface/PositionJointInterface" />
-      <xacro:gazebo-joint joint="${arm_id}_joint6" transmission="hardware_interface/PositionJointInterface" />
-      <xacro:gazebo-joint joint="${arm_id}_joint7" transmission="hardware_interface/PositionJointInterface" />
-      <xacro:gazebo-joint joint="${arm_id}_joint1" transmission="hardware_interface/VelocityJointInterface" />
-      <xacro:gazebo-joint joint="${arm_id}_joint2" transmission="hardware_interface/VelocityJointInterface" />
-      <xacro:gazebo-joint joint="${arm_id}_joint3" transmission="hardware_interface/VelocityJointInterface" />
-      <xacro:gazebo-joint joint="${arm_id}_joint4" transmission="hardware_interface/VelocityJointInterface" />
-      <xacro:gazebo-joint joint="${arm_id}_joint5" transmission="hardware_interface/VelocityJointInterface" />
-      <xacro:gazebo-joint joint="${arm_id}_joint6" transmission="hardware_interface/VelocityJointInterface" />
-      <xacro:gazebo-joint joint="${arm_id}_joint7" transmission="hardware_interface/VelocityJointInterface" />
-      <xacro:gazebo-joint joint="${arm_id}_joint1" transmission="hardware_interface/EffortJointInterface" />
-      <xacro:gazebo-joint joint="${arm_id}_joint2" transmission="hardware_interface/EffortJointInterface" />
-      <xacro:gazebo-joint joint="${arm_id}_joint3" transmission="hardware_interface/EffortJointInterface" />
-      <xacro:gazebo-joint joint="${arm_id}_joint4" transmission="hardware_interface/EffortJointInterface" />
-      <xacro:gazebo-joint joint="${arm_id}_joint5" transmission="hardware_interface/EffortJointInterface" />
-      <xacro:gazebo-joint joint="${arm_id}_joint6" transmission="hardware_interface/EffortJointInterface" />
-      <xacro:gazebo-joint joint="${arm_id}_joint7" transmission="hardware_interface/EffortJointInterface" />
+      <xacro:gazebo-joint joint="${arm_prefix}${arm_id}_joint1" transmission="hardware_interface/PositionJointInterface" />
+      <xacro:gazebo-joint joint="${arm_prefix}${arm_id}_joint2" transmission="hardware_interface/PositionJointInterface" />
+      <xacro:gazebo-joint joint="${arm_prefix}${arm_id}_joint3" transmission="hardware_interface/PositionJointInterface" />
+      <xacro:gazebo-joint joint="${arm_prefix}${arm_id}_joint4" transmission="hardware_interface/PositionJointInterface" />
+      <xacro:gazebo-joint joint="${arm_prefix}${arm_id}_joint5" transmission="hardware_interface/PositionJointInterface" />
+      <xacro:gazebo-joint joint="${arm_prefix}${arm_id}_joint6" transmission="hardware_interface/PositionJointInterface" />
+      <xacro:gazebo-joint joint="${arm_prefix}${arm_id}_joint7" transmission="hardware_interface/PositionJointInterface" />
+      <xacro:gazebo-joint joint="${arm_prefix}${arm_id}_joint1" transmission="hardware_interface/VelocityJointInterface" />
+      <xacro:gazebo-joint joint="${arm_prefix}${arm_id}_joint2" transmission="hardware_interface/VelocityJointInterface" />
+      <xacro:gazebo-joint joint="${arm_prefix}${arm_id}_joint3" transmission="hardware_interface/VelocityJointInterface" />
+      <xacro:gazebo-joint joint="${arm_prefix}${arm_id}_joint4" transmission="hardware_interface/VelocityJointInterface" />
+      <xacro:gazebo-joint joint="${arm_prefix}${arm_id}_joint5" transmission="hardware_interface/VelocityJointInterface" />
+      <xacro:gazebo-joint joint="${arm_prefix}${arm_id}_joint6" transmission="hardware_interface/VelocityJointInterface" />
+      <xacro:gazebo-joint joint="${arm_prefix}${arm_id}_joint7" transmission="hardware_interface/VelocityJointInterface" />
+      <xacro:gazebo-joint joint="${arm_prefix}${arm_id}_joint1" transmission="hardware_interface/EffortJointInterface" />
+      <xacro:gazebo-joint joint="${arm_prefix}${arm_id}_joint2" transmission="hardware_interface/EffortJointInterface" />
+      <xacro:gazebo-joint joint="${arm_prefix}${arm_id}_joint3" transmission="hardware_interface/EffortJointInterface" />
+      <xacro:gazebo-joint joint="${arm_prefix}${arm_id}_joint4" transmission="hardware_interface/EffortJointInterface" />
+      <xacro:gazebo-joint joint="${arm_prefix}${arm_id}_joint5" transmission="hardware_interface/EffortJointInterface" />
+      <xacro:gazebo-joint joint="${arm_prefix}${arm_id}_joint6" transmission="hardware_interface/EffortJointInterface" />
+      <xacro:gazebo-joint joint="${arm_prefix}${arm_id}_joint7" transmission="hardware_interface/EffortJointInterface" />
       <xacro:transmission-franka-state arm_id="${arm_id}" />
       <xacro:transmission-franka-model arm_id="${arm_id}"
-         root="${arm_id}_joint1"
-         tip="${arm_id}_joint8"
+         root="${arm_prefix}${arm_id}_joint1"
+         tip="${arm_prefix}${arm_id}_joint8"
        />
       <xacro:if value="${ee_id == 'franka_hand'}">
-        <xacro:gazebo-joint joint="${arm_id}_finger_joint1" transmission="hardware_interface/EffortJointInterface" />
-        <xacro:gazebo-joint joint="${arm_id}_finger_joint2" transmission="hardware_interface/EffortJointInterface" />
+        <xacro:gazebo-joint joint="${arm_prefix}${arm_id}_finger_joint1" transmission="hardware_interface/EffortJointInterface" />
+        <xacro:gazebo-joint joint="${arm_prefix}${arm_id}_finger_joint2" transmission="hardware_interface/EffortJointInterface" />
         <!-- Friction specific material for Rubber/Rubber contact -->
-        <xacro:gazebo-friction link="${arm_id}_leftfinger" mu="1.13" />
-        <xacro:gazebo-friction link="${arm_id}_rightfinger" mu="1.13" />
+        <xacro:gazebo-friction link="${arm_prefix}${arm_id}_leftfinger" mu="1.13" />
+        <xacro:gazebo-friction link="${arm_prefix}${arm_id}_rightfinger" mu="1.13" />
       </xacro:if>
     </xacro:if>
