Commit message: fix: ee_with_one_link takes the correct arguments

File: robots/common/franka_robot.xacro (robot description, xacro)
@@ -76,6 +76,6 @@
       <xacro:include filename="$(find franka_description)/end_effectors/common/ee_with_one_link.xacro"/>
       <xacro:include filename="$(find franka_description)/end_effectors/common/utils.xacro" />
-      <xacro:property name="special_connection" value="${special_connection}" />
-      <xacro:property name="connection" value="${special_connection if special_connection == '' else arm_id + '_link8'}" />
+      <xacro:property name="special_connection" value="$(arg special_connection)" />
+      <xacro:property name="connection" value="${special_connection if special_connection != '' else arm_id + '_link8'}" />
       <xacro:ee_with_one_link
         connected_to="${arm_prefix}${connection}"
@@ -83,5 +83,5 @@
         arm_prefix="${arm_prefix}"
         ee_id="${ee_id}"
-        ee_inertials="${xacro.load_yaml('$(find franka_description)/end_effectors/${ee_id}/inertials.yaml')}"
+        ee_inertials="${xacro.load_yaml('$(find franka_description)/end_effectors/' + ee_id + '/inertials.yaml')}"
         rpy_ee="${rpy_ee}"
         xyz_ee="${xyz_ee}"

Commit message: fix: remove redundant argument

File: robots/common/franka_robot.xacro (robot description, xacro)
@@ -55,5 +55,4 @@
         <xacro:property name="ee_color" value="white" />
       </xacro:if>
-      <xacro:property name="special_connection" value="$(arg special_connection)" />
       <xacro:property name="connection" value="${special_connection if special_connection != '' else arm_id + '_link8'}" />
       <xacro:franka_hand
@@ -76,5 +75,4 @@
       <xacro:include filename="$(find franka_description)/end_effectors/common/ee_with_one_link.xacro"/>
       <xacro:include filename="$(find franka_description)/end_effectors/common/utils.xacro" />
-      <xacro:property name="special_connection" value="$(arg special_connection)" />
       <xacro:property name="connection" value="${special_connection if special_connection != '' else arm_id + '_link8'}" />
       <xacro:ee_with_one_link
